Commit message: first robot model

File: src/robot_description/urdf/base.xacro (robot description, xacro)
@@ -28,5 +28,5 @@
             </inertial>
             <visual>
-                <origin xyz="0.0 0 ${base_height/2}" rpy="0 0 0" />
+                <origin xyz="0.0 0 0" rpy="0 0 0" />
                 <geometry>
                     <box size="${base_length} ${base_width} ${base_height}" />

File: src/robot_description/urdf/parameter.xacro (robot description, xacro)
@@ -2,12 +2,15 @@
     <xacro:property name="M_PI" value="3.1415926535897931" />
     <!--Chassis Parameter-->
-    <xacro:property name="base_length" value="1.40" /> <!-- value="1.40" -->
-    <xacro:property name="base_width" value="0.705" /> <!-- value="0.705" -->
-    <xacro:property name="base_height" value="0.632" /> <!-- value="0.632" -->
-    <xacro:property name="base_mass" value="25.0" /> <!-- 25 in kg-->
+    <xacro:property name="base_length" value="0.17" /> <!-- value="1.40" -->
+    <xacro:property name="base_width" value="0.10" /> <!-- value="0.705" -->
+    <xacro:property name="base_height" value="0.05" /> <!-- value="0.632" -->
+    <xacro:property name="base_mass" value="0.2" /> <!-- 25 in kg-->
     <!--Wheel Parameter-->
-    <xacro:property name="wheel_radius" value="0.255"/>
-    <xacro:property name="wheel_height" value="0.05" />
-    <xacro:property name="wheel_mass" value="1" /> <!-- 1.5 in kg-->
-    <xacro:property name="track" value="0.62" /> <!--track/2-->
+    <xacro:property name="wheel_radius" value="0.065"/>
+    <xacro:property name="wheel_height" value="0.025" />
+    <xacro:property name="wheel_mass" value="0.050" /> <!-- 1.5 in kg-->
+    <xacro:property name="track" value="0.13" /> <!--track/2-->
+    <xacro:property name="caster_radius" value="0.01"/>
+    <xacro:property name="caster_mass" value="0.01"/>
+    <xacro:property name="caster_dist" value="0.06"/>
 </robot>

File: src/robot_description/urdf/robot.xacro (robot description, xacro)
@@ -11,6 +11,9 @@
 	<!-- import the robot wheel xacro file  -->
 	<xacro:include filename="wheel.xacro" />
+	<xacro:include filename="caster.xacro" />
 	<xacro:robot_base />
 	<xacro:robot_wheel prefix="left" parent="base_link" angle="-1"/>
 	<xacro:robot_wheel prefix="right" parent="base_link" angle="1"/>
+	<xacro:robot_caster prefix="front" parent="base_link" front="1"/>
+	<xacro:robot_caster prefix="back" parent="base_link" front="-1"/>
 </robot>
