Commit message: diff drive imu lidar plugin

File: src/robot_description/urdf/caster.xacro (robot description, xacro)
@@ -29,5 +29,5 @@
       <parent link="${parent}"/>
       <child link="${prefix}_caster"/>
-      <origin xyz="${front*caster_dist} 0 ${-(wheel_radius-caster_radius)+0.001}" rpy="0 0 0" />
+      <origin xyz="${front*caster_dist} 0 ${-(wheel_radius-caster_radius)+0.0001}" rpy="0 0 0" />
     </joint>
   </xacro:macro>

File: src/robot_description/urdf/robot.xacro (robot description, xacro)
@@ -12,4 +12,5 @@
 	<xacro:include filename="wheel.xacro" />
 	<xacro:include filename="caster.xacro" />
+	<xacro:include filename="sensors.xacro" />
 	<xacro:robot_base />
 	<xacro:robot_wheel prefix="left" parent="base_link" angle="-1"/>
@@ -17,3 +18,35 @@
 	<xacro:robot_caster prefix="front" parent="base_link" front="1"/>
 	<xacro:robot_caster prefix="back" parent="base_link" front="-1"/>
+	<xacro:sensor_imu prefix="base" parent="base_link" rate="30"/>
+	<xacro:sensor_2dlidar prefix="base" parent="base_link" rate="30"/>
+	<gazebo>
+	<plugin name='diff_drive' filename='libgazebo_ros_diff_drive.so'>
+		<ros>
+			<!-- Set namespace -->
+			<namespace>/differential_drive_controller</namespace>
+		</ros>
+		<!-- Replace camelCase elements with camel_case ones -->
+		<update_rate>50</update_rate>
+		<left_joint>left_wheel_joint</left_joint>
+		<right_joint>right_wheel_joint</right_joint>
+		<wheel_separation>${track}</wheel_separation>
+		<wheel_diameter>${2*wheel_radius}</wheel_diameter>
+		<odometry_frame>odom</odometry_frame>
+		<!-- wheelTorque and wheelAcceleration now have max_ prefix -->
+		<max_wheel_torque>20</max_wheel_torque>
+		<max_acceleration>1.0</max_acceleration>
+		<!-- output -->
+		<publish_odom>true</publish_odom>
+		<publish_odom_tf>true</publish_odom_tf>
+		<odometry_frame>odom</odometry_frame>
+		<robot_base_frame>base_footprint</robot_base_frame>
+	</plugin>
+	</gazebo>
+	<gazebo>
+		<plugin name="joint_state_publisher" filename="libgazebo_ros_joint_state_publisher.so">
+			<update_rate>2</update_rate>
+			<joint_name>left_wheel_joint</joint_name>
+			<joint_name>right_wheel_joint</joint_name>
+		</plugin>
+	</gazebo>
 </robot>

Commit message: working simulation with noise and slam

File: src/robot_description/urdf/caster.xacro (robot description, xacro)
@@ -26,8 +26,17 @@
       </inertial>
     </link>
+    <gazebo reference="${prefix}_caster">
+      <mu1 value="0.0"/>
+      <mu2 value="0.0"/>
+      <kp  value="10000000.0" />
+      <kd  value="1.0" />
+      <fdir1 value="1 0 0"/>
+      <turnGravityOff>false</turnGravityOff>
+      <minDepth>0.005</minDepth>
+    </gazebo>
     <joint name="${prefix}_caster_joint" type="fixed">
       <parent link="${parent}"/>
       <child link="${prefix}_caster"/>
-      <origin xyz="${front*caster_dist} 0 ${-(wheel_radius-caster_radius)+0.0001}" rpy="0 0 0" />
+      <origin xyz="${front*caster_dist} 0 ${-(wheel_radius-caster_radius)}" rpy="0 0 0" />
     </joint>
   </xacro:macro>

File: src/robot_description/urdf/robot.xacro (robot description, xacro)
@@ -19,31 +19,31 @@
 	<xacro:robot_caster prefix="back" parent="base_link" front="-1"/>
 	<xacro:sensor_imu prefix="base" parent="base_link" rate="30"/>
-	<xacro:sensor_2dlidar prefix="base" parent="base_link" rate="30"/>
+	<xacro:sensor_2dlidar prefix="base" parent="base_link" rate="20"/>
 	<gazebo>
-	<plugin name='diff_drive' filename='libgazebo_ros_diff_drive.so'>
-		<ros>
-			<!-- Set namespace -->
-			<namespace>/differential_drive_controller</namespace>
-		</ros>
-		<!-- Replace camelCase elements with camel_case ones -->
-		<update_rate>50</update_rate>
-		<left_joint>left_wheel_joint</left_joint>
-		<right_joint>right_wheel_joint</right_joint>
-		<wheel_separation>${track}</wheel_separation>
-		<wheel_diameter>${2*wheel_radius}</wheel_diameter>
-		<odometry_frame>odom</odometry_frame>
-		<!-- wheelTorque and wheelAcceleration now have max_ prefix -->
-		<max_wheel_torque>20</max_wheel_torque>
-		<max_acceleration>1.0</max_acceleration>
-		<!-- output -->
-		<publish_odom>true</publish_odom>
-		<publish_odom_tf>true</publish_odom_tf>
-		<odometry_frame>odom</odometry_frame>
-		<robot_base_frame>base_footprint</robot_base_frame>
-	</plugin>
+		<plugin name='diff_drive' filename='libgazebo_ros_diff_drive.so'>
+			<ros>
+				<!-- Set namespace -->
+				<namespace>/differential_drive_controller</namespace>
+			</ros>
+			<!-- Replace camelCase elements with camel_case ones -->
+			<update_rate>50</update_rate>
+			<left_joint>left_wheel_joint</left_joint>
+			<right_joint>right_wheel_joint</right_joint>
+			<wheel_separation>${track}</wheel_separation>
+			<wheel_diameter>${2*wheel_radius}</wheel_diameter>
+			<odometry_frame>odom</odometry_frame>
+			<!-- wheelTorque and wheelAcceleration now have max_ prefix -->
+			<max_wheel_torque>20</max_wheel_torque>
+			<max_acceleration>1.0</max_acceleration>
+			<!-- output -->
+			<publish_odom>true</publish_odom>
+			<publish_odom_tf>true</publish_odom_tf>
+			<odometry_frame>odom</odometry_frame>
+			<robot_base_frame>base_footprint</robot_base_frame>
+		</plugin>
 	</gazebo>
 	<gazebo>
 		<plugin name="joint_state_publisher" filename="libgazebo_ros_joint_state_publisher.so">
-			<update_rate>2</update_rate>
+			<update_rate>50</update_rate>
 			<joint_name>left_wheel_joint</joint_name>
 			<joint_name>right_wheel_joint</joint_name>

File: src/robot_description/urdf/sensors.xacro (robot description, xacro)
@@ -29,5 +29,5 @@
             <always_on>true</always_on>
             <!-- Publish at 30 hz -->
-            <update_rate>30</update_rate>
+            <update_rate>50</update_rate>
             <plugin name="${prefix}_imu" filename="libgazebo_ros_imu_sensor.so">
             <!-- <namespace>/${prefix}_imu</namespace> -->
@@ -66,28 +66,28 @@
         <sensor type="ray" name="${prefix}_2dlidar">
             <ray>
-            <scan>
-                <horizontal>
-                <samples>720</samples>
-                <resolution>1</resolution>
-                <min_angle>${-M_PI}</min_angle>
-                <max_angle>${M_PI}</max_angle>
-                </horizontal>
-            </scan>
-            <range>
-                <min>0.10</min>
-                <max>30.0</max>
-                <resolution>0.01</resolution>
-            </range>
+                <noise>
+                    <type>gaussian</type>
+                    <mean>0.0</mean>
+                    <stddev>0.01</stddev>
+                </noise>
+                <scan>
+                    <horizontal>
+                        <samples>720</samples>
+                        <resolution>1</resolution>
+                        <min_angle>-3.14</min_angle>
+                        <max_angle>3.14</max_angle>
+                    </horizontal>
+                </scan>
+                <range>
+                    <min>0.10</min>
+                    <max>10.0</max>
+                    <resolution>0.03</resolution>
+                </range>
             </ray>
             <always_on>true</always_on>
             <visualize>true</visualize>
             <!-- Using gazebo's update rate instead of plugin's -->
-            <update_rate>30</update_rate>
+            <update_rate>20</update_rate>
             <!-- Using gazebo's noise instead of plugin's -->
-            <noise>
-            <type>gaussian</type>
-            <mean>0.0</mean>
-            <stddev>0.01</stddev>
-            </noise>
             <plugin name="${prefix}_2dlidar" filename="libgazebo_ros_ray_sensor.so">
             <!-- Change namespace and output topic so published topic is /rrbot/laser/scan -->

File: src/robot_description/urdf/wheel.xacro (robot description, xacro)
@@ -33,5 +33,5 @@
       <fdir1 value="1 0 0"/>
       <turnGravityOff>false</turnGravityOff>
-      <!--<minDepth>0.005</minDepth> -->
+      <minDepth>0.005</minDepth>
     </gazebo>
     <joint name="${prefix}_wheel_joint" type="continuous">
